Commit message: added launch file, urdf fixed

File: urdf/lidar.xacro (robot description, xacro)
@@ -1,5 +1,5 @@
 <?xml version="1.0"?>
 <robot xmlns:xacro="http://www.ros.org/wiki/xacro">
-  <link name="lidar">
+  <link name="laser">
     <visual>
       <geometry>
@@ -19,5 +19,5 @@
   <joint name="lidar_joint" type="fixed">
     <parent link="base_link"/>
-    <child link="lidar"/>
+    <child link="laser"/>
     <origin xyz="-0.052 -0.2 0.0325"/>
   </joint>
